File: main/_autosave-main.sch (KiCad schematic (older format))
At the start: 35 parts, among them J1 Conn_01x10_Female, J2 USB_B, J3 AVR-ISP-6, J4 Micro SD Card, Q1 2N7002, Q2 BSS84, U1 ATmega1284P-PU, U2 AMS1117, U3 MCP2221A-I_SL, U4 TXB0104D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

Commit message: fixed layout
Parts:
- renumbered Reset to SW1
Changed lines of the file:
@@
 RST
 $Comp
-L Switch:SW_Push Reset
+L Switch:SW_Push SW1
 U 1 1 6941B491
 P 4650 2050
-F 0 "Reset" H 4650 2335 50  0000 C CNN
+F 0 "SW1" H 4650 2335 50  0000 C CNN
 F 1 "SW1" H 4650 2244 50  0000 C CNN
 F 2 "Button_Switch_SMD:SW_SPST_B3SL-1002P" H 4650 2250 50  0001 C CNN
