File: main/main.kicad_pcb (KiCad board)
At the start: 4 copper layers, 72.5 x 60 mm, 35 parts, among them J1 Conn_01x10_Female, J2 USB_B, J3 AVR-ISP-6, J4 Micro_SD_Card, Q1 2N7002, Q2 BSS84, SW1 Reset, U1 ATmega1284P-PU, U2 AMS1117, U3 MCP2221A-I_SL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

Commit message: fixed layout
Parts:
- J4: value Micro_SD_Card -> Micro SD Card; footprint footprints:5033981892 -> footprints:5027740891
- SW1: value Reset -> SW1
- moved J2 1.50 mm to (73.0, 120.8)
- moved C7 1.46 mm to (80.0, 122.0), turned to 270 degrees
- moved J4 1.06 mm to (66.0, 101.8), turned to 90 degrees
Routing:
- net SD_CS: track 33.3 -> 42.3 mm
- net D-: track 22.3 -> 24.7 mm
- net +3V3: track 83.7 -> 85.7 mm
- net D+: track 24.7 -> 26.2 mm
- net GND: track 51.9 -> 53.4 mm
- net SD_MOSI: track 22.6 -> 21.6 mm
- net SD_MISO: track 25.3 -> 24.2 mm
Other:
- board text added: "Reset"
